File: hardware/template.kicad_pcb (KiCad board)
At the start: 4 copper layers, 105 x 75 mm, 82 parts, among them IC1 AG9912M, IC2 RTL8201F-VB-CG, IC3 SY8120B1ABC, J1 JXD1-0009NL, J2 SHF-108-01-L-D-SM, J3 SHF-103-01-L-D-SM, SW1 SW_Push, U1 PAC1932T-I/JQ, U2 ESP32-WROVER-E-N4R8, U3 PCA9536TK, X1 SG-5032CCN

Commit message: test
Parts:
- moved J3 2.17 mm to (111.0, 94.1)
Routing:
- net /mcu/esp32/RXD0: track 4.41 -> 6.68 mm
- net /mcu/esp32/TXD0: track 4.41 -> 6.68 mm
- net /mcu/ESP_EN: track 92.8 -> 94.3 mm
- net /mcu/+3.3V: track 60.7 -> 61.9 mm
- net /mcu/GPIO0: track 72.4 -> 73.6 mm
- net /mcu/GND: vias 90 -> 89

Commit message: test_2
Parts:
- moved J3 10.7 mm to (117.3, 85.5)
Changed lines of the file:
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@@
   )
   (footprint "general:SAMTEC_SHF-103-01-L-D-SM" (layer "F.Cu")
-    (at 110.998 94.107)
+    (at 117.348 85.4705)
     (property "MANUFACTURER" "Samtec")
     (property "Manufacturer_Part_Number" "SHF-103-01-L-D-SM")

Commit message: new
Parts:
- moved J3 15.6 mm to (132.6, 82.3)
Changed lines of the file:
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@@
   )
   (footprint "general:SAMTEC_SHF-103-01-L-D-SM" (layer "F.Cu")
-    (at 117.348 85.4705)
+    (at 132.588 82.2965)
     (property "MANUFACTURER" "Samtec")
     (property "Manufacturer_Part_Number" "SHF-103-01-L-D-SM")
